File: Hardware/v1/USB-Meter.sch (KiCad schematic (older format))
At the start: 80 parts, among them J1 Screw_Terminal_01x02, J12 Conn_01x02, J13 Conn_01x02, J14 Conn_ARM_JTAG_SWD_10, J2 USB_B_Micro, J3 USB_A, J6 Conn_02x04_Odd_Even, J9 Conn_02x04_Odd_Even, SW2 SW_Push, SW3 SW_Push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

Commit message: Fix schematic library refs
Parts:
- J2: symbol Connector:USB_B_Micro -> USB-Meter-rescue:USB_B_Micro-Connector
- J3: symbol Connector:USB_A -> USB-Meter-rescue:USB_A-Connector
- U2: symbol Regulator_Linear:AP2127K-3.3 -> USB-Meter-rescue:AP2127K-3.3-Regulator_Linear
- U3, U4: symbol Power_Protection:USBLC6-2SC6 -> USB-Meter-rescue:USBLC6-2SC6-Power_Protection
Changed lines of the file:
@@
 EESchema Schematic File Version 4
-LIBS:USB-Meter-cache
 EELAYER 30 0
 EELAYER END
@@
 $EndDescr
 $Comp
-L Connector:USB_A J3
+L USB-Meter-rescue:USB_A-Connector J3
 U 1 1 5C23E990
 P 14700 2450
@@
 D_HOST-
 $Comp
-L Regulator_Linear:AP2127K-3.3 U2
+L USB-Meter-rescue:AP2127K-3.3-Regulator_Linear U2
 U 1 1 5C244B64
 P 4700 5000
@@
 VEXT_DET_CTRL
 $Comp
-L Connector:USB_B_Micro J2
+L USB-Meter-rescue:USB_B_Micro-Connector J2
 U 1 1 5CF47233
 P 1550 7550
@@
 GND_CTRL
 $Comp
-L Power_Protection:USBLC6-2SC6 U3
+L USB-Meter-rescue:USBLC6-2SC6-Power_Protection U3
 U 1 1 5DD22C7E
 P 4150 7600
@@
 $EndComp
 $Comp
-L Power_Protection:USBLC6-2SC6 U4
+L USB-Meter-rescue:USBLC6-2SC6-Power_Protection U4
 U 1 1 5DD4FF01
 P 12550 2450
